File: AppleIIJoystick.sch (KiCad schematic (older format))
At the start: 4 parts

Commit message: finished schematic
Parts:
- added C? (x6): C, symbol Device:C
- added R? (x2): 220, symbol Device:R
- added R? (x2): 560, symbol Device:R
- added RV?: R_POT_TRIM, symbol Device:R_POT_TRIM
Connections:
- net PB1: now reaches J?.1
- net PB1: now also SW?.2, R?.1
- net +5V: now reaches J?.2
- net +5V: now also J?.2 (LR), J?.3 (UD), J?.6 (UD), J?.7 (LR), SW?.1, SW?.1
- net GND: now reaches J?.3
- net GND: now also C?.2, C?.2, C?.2, C?.2, C?.2, C?.2, R?.2, R?.2
- net LR: now reaches J?.5
- net LR: now also C?.1, C?.1, C?.1, R?.2
- net PB0: now reaches J?.7
- net PB0: now also SW?.2, R?.1
- net UD: now reaches J?.8
- net UD: now also C?.1, C?.1, C?.1, R?.2
- net at J?.1 (LR+): now also R?.1
- net at J?.8 (UD+): now also R?.1
- no-connect marks 0 -> 5
Other:
- moved on the sheet: J?, SW?

Commit message: starting footprint/3d models
Parts:
- removed RV?: R_POT_TRIM, symbol Device:R_POT_TRIM
- added C4: 10nF, symbol Device:C
- added C5: .1uF, symbol Device:C
- added R1, R4: RTRIM, symbol Device:RTRIM
- C1, C2, C3, C6, C7: renamed from C?; value C -> .1uF
- C8: renamed from C?; value C -> 10nF
- R2, R3: renamed from R?; value 220 -> 180
- gave numbers to parts that had none: 6
Connections:
- net GND: now also C4.2, C5.2
- net LR: now also C4.1, R1.2; no longer R2.2
- net UD: now also C5.1, R4.1; no longer R3.2
- new net: R1.1, R2.2
- new net: R3.2, R4.2
Changed lines of the file:
@@
 $EndDescr
 $Comp
-L Connector:DB9_Male J?
+L Connector:DB9_Male J1
 U 1 1 5DC4324C
 P 1570 3425
-F 0 "J?" H 1488 2733 50  0000 C CNN
+F 0 "J1" H 1488 2733 50  0000 C CNN
 F 1 "DB9_Male" H 1488 2824 50  0000 C CNN
 F 2 "" H 1570 3425 50  0001 C CNN
@@
 $EndComp
 $Comp
-L AppleIIJoystick:Parallax_27800_Joystick J?
+L AppleIIJoystick:Parallax_27800_Joystick J2
 U 1 1 5DC45FAC
 P 6515 3510
-F 0 "J?" H 6515 4185 50  0000 C CNN
+F 0 "J2" H 6515 4185 50  0000 C CNN
 F 1 "Parallax_27800_Joystick" H 6515 4094 50  0000 C CNN
 F 2 "" H 6565 3460 50  0001 C CNN
@@
 $EndComp
 $Comp
-L Switch:SW_Push SW?
+L Switch:SW_Push SW1
 U 1 1 5DC52EB7
 P 8575 4860
-F 0 "SW?" H 8575 5145 50  0000 C CNN
+F 0 "SW1" H 8575 5145 50  0000 C CNN
 F 1 "SW_Push" H 8575 5054 50  0000 C CNN
 F 2 "" H 8575 5060 50  0001 C CNN
@@
 $EndComp
 $Comp
-L Switch:SW_Push SW?
+L Switch:SW_Push SW2
 U 1 1 5DC533F1
 P 8575 5720
-F 0 "SW?" H 8575 6005 50  0000 C CNN
+F 0 "SW2" H 8575 6005 50  0000 C CNN
 F 1 "SW_Push" H 8575 5914 50  0000 C CNN
 F 2 "" H 8575 5920 50  0001 C CNN
@@
 	5620 3060 5865 3060
 $Comp
-L Device:R R?
+L Device:R R2
 U 1 1 5DC582DF
 P 5470 3060
-F 0 "R?" V 5263 3060 50  0000 C CNN
-F 1 "220" V 5470 3060 50  0000 C CNN
+F 0 "R2" V 5263 3060 50  0000 C CNN
+F 1 "180" V 5470 3060 50  0000 C CNN
 F 2 "" V 5400 3060 50  0001 C CNN
 F 3 "~" H 5470 3060 50  0001 C CNN
@@
 	7410 3060 7165 3060
 $Comp
-L Device:R R?
+L Device:R R3
 U 1 1 5DC5961D
 P 7560 3060
-F 0 "R?" V 7353 3060 50  0000 C CNN
-F 1 "220" V 7560 3060 50  0000 C CNN
+F 0 "R3" V 7353 3060 50  0000 C CNN
+F 1 "180" V 7560 3060 50  0000 C CNN
 F 2 "" V 7490 3060 50  0001 C CNN
 F 3 "~" H 7560 3060 50  0001 C CNN
@@
 +5V
 $Comp
-L Device:R R?
+L Device:R R5
 U 1 1 5DC5A8EF
 P 8930 5080
-F 0 "R?" V 8723 5080 50  0000 C CNN
+F 0 "R5" V 8723 5080 50  0000 C CNN
 F 1 "560" V 8930 5080 50  0000 C CNN
 F 2 "" V 8860 5080 50  0001 C CNN
@@
 	8930 5230 8930 5325
 $Comp
-L power:GND #PWR?
+L power:GND #PWR04
 U 1 1 5DC5B58B
 P 8930 5325
-F 0 "#PWR?" H 8930 5075 50  0001 C CNN
+F 0 "#PWR04" H 8930 5075 50  0001 C CNN
 F 1 "GND" H 8935 5152 50  0000 C CNN
 F 2 "" H 8930 5325 50  0001 C CNN
@@
 +5V
 $Comp
-L Device:R R?
+L Device:R R6
 U 1 1 5DC5D1C7
 P 8930 5940
-F 0 "R?" V 8723 5940 50  0000 C CNN
+F 0 "R6" V 8723 5940 50  0000 C CNN
 F 1 "560" V 8930 5940 50  0000 C CNN
 F 2 "" V 8860 5940 50  0001 C CNN
@@
 Wire Wire Line
 	8930 5720 8775 5720
-Wire Wire Line
-	8930 6090 8930 6185
-$Comp
-L power:GND #PWR?
+$Comp
+L power:GND #PWR05
 U 1 1 5DC5D1D0
 P 8930 6185
-F 0 "#PWR?" H 8930 5935 50  0001 C CNN
+F 0 "#PWR05" H 8930 5935 50  0001 C CNN
 F 1 "GND" H 8935 6012 50  0000 C CNN
 F 2 "" H 8930 6185 50  0001 C CNN
@@
 PB0
 $Comp
-L Device:C C?
+L Device:C C6
 U 1 1 5DC5D4FD
 P 8155 3450
-F 0 "C?" H 8270 3496 50  0000 L CNN
-F 1 "C" H 8270 3405 50  0000 L CNN
+F 0 "C6" H 8155 3525 50  0000 L CNN
+F 1 ".1uF" H 8155 3370 50  0000 L CNN
 F 2 "" H 8193 3300 50  0001 C CNN
 F 3 "~" H 8155 3450 50  0001 C CNN
@@
 $EndComp
 $Comp
-L Device:C C?
+L Device:C C7
 U 1 1 5DC5D8A6
 P 8460 3450
-F 0 "C?" H 8575 3496 50  0000 L CNN
-F 1 "C" H 8575 3405 50  0000 L CNN
+F 0 "C7" H 8460 3525 50  0000 L CNN
+F 1 ".1uF" H 8460 3375 50  0000 L CNN
 F 2 "" H 8498 3300 50  0001 C CNN
 F 3 "~" H 8460 3450 50  0001 C CNN
@@
 $EndComp
 $Comp
-L Device:C C?
+L Device:C C8
 U 1 1 5DC5DF0E
 P 8780 3450
-F 0 "C?" H 8895 3496 50  0000 L CNN
-F 1 "C" H 8895 3405 50  0000 L CNN
+F 0 "C8" H 8780 3525 50  0000 L CNN
+F 1 "10nF" H 8780 3375 50  0000 L CNN
 F 2 "" H 8818 3300 50  0001 C CNN
 F 3 "~" H 8780 3450 50  0001 C CNN
@@
 	8460 3710 8460 3785
 $Comp
-L power:GND #PWR?
+L power:GND #PWR03
 U 1 1 5DC5EDD1
 P 8460 3785
-F 0 "#PWR?" H 8460 3535 50  0001 C CNN
+F 0 "#PWR03" H 8460 3535 50  0001 C CNN
 F 1 "GND" H 8465 3612 50  0000 C CNN
 F 2 "" H 8460 3785 50  0001 C CNN
@@
 	8460 3175 8460 3060
 Wire Wire Line
-	8460 3060 7710 3060
-Wire Wire Line
 	8460 3060 8690 3060
-Connection ~ 8460 3060
 Text Label 8690 3060 2    50   ~ 0
 UD
 $Comp
-L Device:C C?
-U 1 1 5DC611C1
-P 4875 3450
-F 0 "C?" H 4990 3496 50  0000 L CNN
-F 1 "C" H 4990 3405 50  0000 L CNN
-F 2 "" H 4913 3300 50  0001 C CNN
-F 3 "~" H 4875 3450 50  0001 C CNN
-	1    4875 3450
-	-1   0    0    -1
-$EndComp
-$Comp
-L Device:C C?
-U 1 1 5DC611CB
-P 4570 3450
-F 0 "C?" H 4685 3496 50  0000 L CNN
-F 1 "C" H 4685 3405 50  0000 L CNN
-F 2 "" H 4608 3300 50  0001 C CNN
-F 3 "~" H 4570 3450 50  0001 C CNN
-	1    4570 3450
-	-1   0    0    -1
-$EndComp
-$Comp
-L Device:C C?
+L Device:C C1
 U 1 1 5DC611D5
 P 4250 3450
-F 0 "C?" H 4365 3496 50  0000 L CNN
-F 1 "C" H 4365 3405 50  0000 L CNN
+F 0 "C1" H 4250 3525 50  0000 R CNN
+F 1 ".1uF" H 4250 3370 50  0000 R CNN
 F 2 "" H 4288 3300 50  0001 C CNN
 F 3 "~" H 4250 3450 50  0001 C CNN
@@
 	4570 3710 4570 3785
 $Comp
-L power:GND #PWR?
+L power:GND #PWR02
 U 1 1 5DC611E6
 P 4570 3785
-F 0 "#PWR?" H 4570 3535 50  0001 C CNN
+F 0 "#PWR02" H 4570 3535 50  0001 C CNN
 F 1 "GND" H 4575 3612 50  0000 C CNN
 F 2 "" H 4570 3785 50  0001 C CNN
@@
 	4570 3175 4570 3060
 Wire Wire Line
-	4570 3060 5320 3060
-Wire Wire Line
 	4570 3060 4340 3060
-Connection ~ 4570 3060
 Text Label 4340 3060 0    50   ~ 0
 LR
@@
 	1870 3425 2145 3425
 $Comp
-L power:GND #PWR?
+L power:GND #PWR01
 U 1 1 5DC6EA63
 P 2145 3425
-F 0 "#PWR?" H 2145 3175 50  0001 C CNN
+F 0 "#PWR01" H 2145 3175 50  0001 C CNN
 F 1 "GND" V 2150 3297 50  0000 R CNN
 F 2 "" H 2145 3425 50  0001 C CNN
@@
 NoConn ~ 1870 3125
 $Comp
-L Device:R_POT_TRIM RV?
-U 1 1 5DC73122
-P 4945 2680
-F 0 "RV?" H 4875 2726 50  0000 R CNN
-F 1 "R_POT_TRIM" H 4875 2635 50  0000 R CNN
-F 2 "" H 4945 2680 50  0001 C CNN
-F 3 "~" H 4945 2680 50  0001 C CNN
-	1    4945 2680
-	1    0    0    -1
-$EndComp
+L Device:C C4
+U 1 1 5DC739E9
+P 5180 3450
+F 0 "C4" H 5075 3525 50  0000 L CNN
+F 1 "10nF" H 4990 3370 50  0000 L CNN
+F 2 "" H 5218 3300 50  0001 C CNN
+F 3 "~" H 5180 3450 50  0001 C CNN
+	1    5180 3450
+	-1   0    0    -1
+$EndComp
+Wire Wire Line
+	5180 3300 5180 3175
+Wire Wire Line
+	5180 3175 4875 3175
+Connection ~ 4875 3175
+Wire Wire Line
+	5180 3600 5180 3710
+Wire Wire Line
+	5180 3710 4875 3710
+Connection ~ 4875 3710
+$Comp
+L Device:C C5
+U 1 1 5DC82559
+P 7850 3450
+F 0 "C5" H 7850 3525 50  0000 L CNN
+F 1 ".1uF" H 7850 3380 50  0000 L CNN
+F 2 "" H 7888 3300 50  0001 C CNN
+F 3 "~" H 7850 3450 50  0001 C CNN
+	1    7850 3450
+	1    0    0    -1
+$EndComp
+Wire Wire Line
+	7850 3600 7850 3710
+Wire Wire Line
+	7850 3175 7850 3300
+Wire Wire Line
+	8155 3175 7850 3175
+Connection ~ 8155 3175
+Wire Wire Line
+	7850 3710 8155 3710
+Connection ~ 8155 3710
+$Comp
+L Device:C C3
+U 1 1 5DC611C1
+P 4875 3450
+F 0 "C3" H 4780 3525 50  0000 L CNN
+F 1 ".1uF" H 4710 3370 50  0000 L CNN
+F 2 "" H 4913 3300 50  0001 C CNN
+F 3 "~" H 4875 3450 50  0001 C CNN
+	1    4875 3450
+	-1   0    0    -1
+$EndComp
+$Comp
+L Device:C C2
+U 1 1 5DC611CB
+P 4570 3450
+F 0 "C2" H 4470 3525 50  0000 L CNN
+F 1 ".1uF" H 4405 3365 50  0000 L CNN
+F 2 "" H 4608 3300 50  0001 C CNN
+F 3 "~" H 4570 3450 50  0001 C CNN
+	1    4570 3450
+	-1   0    0    -1
+$EndComp
+$Comp
+L Device:RTRIM R1
+U 1 1 5DC87432
+P 5000 3060
+F 0 "R1" V 4760 3060 50  0000 C CNN
+F 1 "RTRIM" V 4851 3060 50  0000 C CNN
+F 2 "" V 4930 3060 50  0001 C CNN
+F 3 "~" H 5000 3060 50  0001 C CNN
+	1    5000 3060
+	0    1    1    0
+$EndComp
+Wire Wire Line
+	5150 3060 5320 3060
+Wire Wire Line
+	4850 3060 4570 3060
+Connection ~ 4570 3060
+$Comp
+L Device:RTRIM R4
+U 1 1 5DC8A203
+P 8085 3060
+F 0 "R4" V 7845 3060 50  0000 C CNN
+F 1 "RTRIM" V 7936 3060 50  0000 C CNN
+F 2 "" V 8015 3060 50  0001 C CNN
+F 3 "~" H 8085 3060 50  0001 C CNN
+	1    8085 3060
+	0    1    1    0
+$EndComp
+Wire Wire Line
+	7935 3060 7710 3060
+Wire Wire Line
+	8235 3060 8460 3060
+Connection ~ 8460 3060
+Wire Wire Line
+	8930 6090 8930 6185
 $EndSCHEMATC

Commit message: db9 footprint/3d model created
Parts:
- C1, C2, C3, C4, C5, C6, C7, C8: footprint (none) -> Capacitor_THT:C_Disc_D3.0mm_W2.0mm_P2.50mm
- J2: footprint (none) -> AppleIIJoystick:Parallax_27800_Joystick
- R2, R3, R5, R6: footprint (none) -> Resistor_THT:R_Axial_DIN0207_L6.3mm_D2.5mm_P10.16mm_Horizontal
- SW1, SW2: footprint (none) -> AppleIIJoystick:D6C_BUTTON
Changed lines of the file:
@@
 F 0 "J2" H 6515 4185 50  0000 C CNN
 F 1 "Parallax_27800_Joystick" H 6515 4094 50  0000 C CNN
-F 2 "" H 6565 3460 50  0001 C CNN
+F 2 "AppleIIJoystick:Parallax_27800_Joystick" H 6565 3460 50  0001 C CNN
 F 3 "" H 6565 3460 50  0001 C CNN
 	1    6515 3510
@@
 F 0 "SW1" H 8575 5145 50  0000 C CNN
 F 1 "SW_Push" H 8575 5054 50  0000 C CNN
-F 2 "" H 8575 5060 50  0001 C CNN
+F 2 "AppleIIJoystick:D6C_BUTTON" H 8575 5060 50  0001 C CNN
 F 3 "~" H 8575 5060 50  0001 C CNN
 	1    8575 4860
@@
 F 0 "SW2" H 8575 6005 50  0000 C CNN
 F 1 "SW_Push" H 8575 5914 50  0000 C CNN
-F 2 "" H 8575 5920 50  0001 C CNN
+F 2 "AppleIIJoystick:D6C_BUTTON" H 8575 5920 50  0001 C CNN
 F 3 "~" H 8575 5920 50  0001 C CNN
 	1    8575 5720
@@
 F 0 "R2" V 5263 3060 50  0000 C CNN
 F 1 "180" V 5470 3060 50  0000 C CNN
-F 2 "" V 5400 3060 50  0001 C CNN
+F 2 "Resistor_THT:R_Axial_DIN0207_L6.3mm_D2.5mm_P10.16mm_Horizontal" V 5400 3060 50  0001 C CNN
 F 3 "~" H 5470 3060 50  0001 C CNN
 	1    5470 3060
@@
 F 0 "R3" V 7353 3060 50  0000 C CNN
 F 1 "180" V 7560 3060 50  0000 C CNN
-F 2 "" V 7490 3060 50  0001 C CNN
+F 2 "Resistor_THT:R_Axial_DIN0207_L6.3mm_D2.5mm_P10.16mm_Horizontal" V 7490 3060 50  0001 C CNN
 F 3 "~" H 7560 3060 50  0001 C CNN
 	1    7560 3060
@@
 F 0 "R5" V 8723 5080 50  0000 C CNN
 F 1 "560" V 8930 5080 50  0000 C CNN
-F 2 "" V 8860 5080 50  0001 C CNN
+F 2 "Resistor_THT:R_Axial_DIN0207_L6.3mm_D2.5mm_P10.16mm_Horizontal" V 8860 5080 50  0001 C CNN
 F 3 "~" H 8930 5080 50  0001 C CNN
 	1    8930 5080
@@
 F 0 "R6" V 8723 5940 50  0000 C CNN
 F 1 "560" V 8930 5940 50  0000 C CNN
-F 2 "" V 8860 5940 50  0001 C CNN
+F 2 "Resistor_THT:R_Axial_DIN0207_L6.3mm_D2.5mm_P10.16mm_Horizontal" V 8860 5940 50  0001 C CNN
 F 3 "~" H 8930 5940 50  0001 C CNN
 	1    8930 5940
@@
 F 0 "C6" H 8155 3525 50  0000 L CNN
 F 1 ".1uF" H 8155 3370 50  0000 L CNN
-F 2 "" H 8193 3300 50  0001 C CNN
+F 2 "Capacitor_THT:C_Disc_D3.0mm_W2.0mm_P2.50mm" H 8193 3300 50  0001 C CNN
 F 3 "~" H 8155 3450 50  0001 C CNN
 	1    8155 3450
@@
 F 0 "C7" H 8460 3525 50  0000 L CNN
 F 1 ".1uF" H 8460 3375 50  0000 L CNN
-F 2 "" H 8498 3300 50  0001 C CNN
+F 2 "Capacitor_THT:C_Disc_D3.0mm_W2.0mm_P2.50mm" H 8498 3300 50  0001 C CNN
 F 3 "~" H 8460 3450 50  0001 C CNN
 	1    8460 3450
@@
 F 0 "C8" H 8780 3525 50  0000 L CNN
 F 1 "10nF" H 8780 3375 50  0000 L CNN
-F 2 "" H 8818 3300 50  0001 C CNN
+F 2 "Capacitor_THT:C_Disc_D3.0mm_W2.0mm_P2.50mm" H 8818 3300 50  0001 C CNN
 F 3 "~" H 8780 3450 50  0001 C CNN
 	1    8780 3450
@@
 F 0 "C1" H 4250 3525 50  0000 R CNN
 F 1 ".1uF" H 4250 3370 50  0000 R CNN
-F 2 "" H 4288 3300 50  0001 C CNN
+F 2 "Capacitor_THT:C_Disc_D3.0mm_W2.0mm_P2.50mm" H 4288 3300 50  0001 C CNN
 F 3 "~" H 4250 3450 50  0001 C CNN
 	1    4250 3450
@@
 F 0 "C4" H 5075 3525 50  0000 L CNN
 F 1 "10nF" H 4990 3370 50  0000 L CNN
-F 2 "" H 5218 3300 50  0001 C CNN
+F 2 "Capacitor_THT:C_Disc_D3.0mm_W2.0mm_P2.50mm" H 5218 3300 50  0001 C CNN
 F 3 "~" H 5180 3450 50  0001 C CNN
 	1    5180 3450
@@
 F 0 "C5" H 7850 3525 50  0000 L CNN
 F 1 ".1uF" H 7850 3380 50  0000 L CNN
-F 2 "" H 7888 3300 50  0001 C CNN
+F 2 "Capacitor_THT:C_Disc_D3.0mm_W2.0mm_P2.50mm" H 7888 3300 50  0001 C CNN
 F 3 "~" H 7850 3450 50  0001 C CNN
 	1    7850 3450
@@
 F 0 "C3" H 4780 3525 50  0000 L CNN
 F 1 ".1uF" H 4710 3370 50  0000 L CNN
-F 2 "" H 4913 3300 50  0001 C CNN
+F 2 "Capacitor_THT:C_Disc_D3.0mm_W2.0mm_P2.50mm" H 4913 3300 50  0001 C CNN
 F 3 "~" H 4875 3450 50  0001 C CNN
 	1    4875 3450
@@
 F 0 "C2" H 4470 3525 50  0000 L CNN
 F 1 ".1uF" H 4405 3365 50  0000 L CNN
-F 2 "" H 4608 3300 50  0001 C CNN
+F 2 "Capacitor_THT:C_Disc_D3.0mm_W2.0mm_P2.50mm" H 4608 3300 50  0001 C CNN
 F 3 "~" H 4570 3450 50  0001 C CNN
 	1    4570 3450

Commit message: added x,y trim pot and imported net list
Parts:
- J1: footprint (none) -> AppleIIJoystick:ADS09_DB9
- R1, R4: footprint (none) -> AppleIIJoystick:PT10LV10_TRIM_POT
- SW1, SW2: symbol Switch:SW_Push -> AppleIIJoystick:SW_Push
Connections:
- net PB0: now also SW2.3; no longer SW2.2
- net PB1: now also SW1.3; no longer SW1.2
Changed lines of the file:
@@
 F 0 "J1" H 1488 2733 50  0000 C CNN
 F 1 "DB9_Male" H 1488 2824 50  0000 C CNN
-F 2 "" H 1570 3425 50  0001 C CNN
+F 2 "AppleIIJoystick:ADS09_DB9" H 1570 3425 50  0001 C CNN
 F 3 " ~" H 1570 3425 50  0001 C CNN
 	1    1570 3425
@@
 $EndComp
 $Comp
-L Switch:SW_Push SW1
+L AppleIIJoystick:SW_Push SW1
 U 1 1 5DC52EB7
 P 8575 4860
@@
 $EndComp
 $Comp
-L Switch:SW_Push SW2
+L AppleIIJoystick:SW_Push SW2
 U 1 1 5DC533F1
 P 8575 5720
@@
 F 0 "R1" V 4760 3060 50  0000 C CNN
 F 1 "RTRIM" V 4851 3060 50  0000 C CNN
-F 2 "" V 4930 3060 50  0001 C CNN
+F 2 "AppleIIJoystick:PT10LV10_TRIM_POT" V 4930 3060 50  0001 C CNN
 F 3 "~" H 5000 3060 50  0001 C CNN
 	1    5000 3060
@@
 F 0 "R4" V 7845 3060 50  0000 C CNN
 F 1 "RTRIM" V 7936 3060 50  0000 C CNN
-F 2 "" V 8015 3060 50  0001 C CNN
+F 2 "AppleIIJoystick:PT10LV10_TRIM_POT" V 8015 3060 50  0001 C CNN
 F 3 "~" H 8085 3060 50  0001 C CNN
 	1    8085 3060

Commit message: swapped out buttons. new footprint/3d model.
Parts:
- SW1, SW2: footprint AppleIIJoystick:D6C_BUTTON -> AppleIIJoystick:ESWITCH_E11GRY_BTN
Changed lines of the file:
@@
 F 0 "SW1" H 8575 5145 50  0000 C CNN
 F 1 "SW_Push" H 8575 5054 50  0000 C CNN
-F 2 "AppleIIJoystick:D6C_BUTTON" H 8575 5060 50  0001 C CNN
+F 2 "AppleIIJoystick:ESWITCH_E11GRY_BTN" H 8575 5060 50  0001 C CNN
 F 3 "~" H 8575 5060 50  0001 C CNN
 	1    8575 4860
@@
 F 0 "SW2" H 8575 6005 50  0000 C CNN
 F 1 "SW_Push" H 8575 5914 50  0000 C CNN
-F 2 "AppleIIJoystick:D6C_BUTTON" H 8575 5920 50  0001 C CNN
+F 2 "AppleIIJoystick:ESWITCH_E11GRY_BTN" H 8575 5920 50  0001 C CNN
 F 3 "~" H 8575 5920 50  0001 C CNN
 	1    8575 5720

Commit message: board layout
Connections:
- net LR: now also R1.1; no longer R1.2
- net at R2.2: now also R1.2; no longer R1.1
Other:
- moved on the sheet: R1
Changed lines of the file:
@@
 U 1 1 5DC87432
 P 5000 3060
-F 0 "R1" V 4760 3060 50  0000 C CNN
-F 1 "RTRIM" V 4851 3060 50  0000 C CNN
+F 0 "R1" V 5265 3060 50  0000 C CNN
+F 1 "RTRIM" V 5174 3060 50  0000 C CNN
 F 2 "AppleIIJoystick:PT10LV10_TRIM_POT" V 4930 3060 50  0001 C CNN
 F 3 "~" H 5000 3060 50  0001 C CNN
 	1    5000 3060
-	0    1    1    0
+	0    -1   -1   0
 $EndComp
 Wire Wire Line
